Commit message: Added Wolverbot URDF

File: src/bitbots_robot/wolfgang_description/urdf/robot.urdf (robot description, URDF)
Before this commit: robot wolfgang, 48 links, 47 joints
Links:
- removed link base_link
- removed link camera
- removed link camera_optical_frame_uncalibrated
- removed link head
- removed link imu_frame_2
- removed link imu_frame_uncalibrated
- removed link l_ankle
- removed link l_cleat_l_back
- removed link l_cleat_l_front
- removed link l_cleat_r_back
- removed link l_cleat_r_front
- removed link l_foot
- removed link l_hip_1
- removed link l_hip_2
- removed link l_lower_arm
- removed link l_lower_leg
- removed link l_shoulder
- removed link l_sole
- removed link l_toe
- removed link l_upper_arm
- removed link l_upper_leg
- removed link l_wrist
- removed link llb
- removed link llf
- removed link lrb
- removed link lrf
- removed link neck
- removed link r_ankle
- removed link r_cleat_l_back
- removed link r_cleat_l_front
- removed link r_cleat_r_back
- removed link r_cleat_r_front
- removed link r_foot
- removed link r_hip_1
- removed link r_hip_2
- removed link r_lower_arm
- removed link r_lower_leg
- removed link r_shoulder
- removed link r_sole
- removed link r_toe
- removed link r_upper_arm
- removed link r_upper_leg
- removed link r_wrist
- removed link rlb
- removed link rlf
- removed link rrb
- removed link rrf
- added link 60645k191_ball_joint_rod_end, mass 0.00402112; visual mesh filename=package://assets/60645k191_ball_joint_rod_end.stl
- added link 60645k191_ball_joint_rod_end_2, mass 0.00402112; visual mesh filename=package://assets/60645k191_ball_joint_rod_end.stl
- added link head_bottom, mass 0.0175792; visual mesh filename=package://assets/head_bottom.stl
- added link head_top, mass 0.107163; visual mesh filename=package://assets/head_top.stl
- added link hip_left_x, mass 0.0526167; visual mesh filename=package://assets/hip_left_x.stl
- added link hip_left_z, mass 0.0517715; collision box size=0.0311905 0.00586106 0.034; collision box size=0.0317858 0.0071103 0.034
- added link hip_right_x, mass 0.0526167; visual mesh filename=package://assets/hip_right_x.stl
- added link hip_right_z, mass 0.0517715; collision box size=0.0311905 0.00586106 0.034; collision box size=0.0317858 0.0071103 0.034
- added link left_arm, mass 0.121563; collision box size=0.029846 0.205415 0.048; visual mesh filename=package://assets/left_arm.stl
- added link left_foot, mass 0.132264; collision box size=0.0399948 0.0108051 0.01; collision box size=0.061605 0.0990193 0.01
- added link left_hand, mass 0.146964; collision box size=0.0319403 0.0740559 0.041; collision box size=0.032 0.0302663 0.041
- added link left_shin, mass 0.363327; visual mesh filename=package://assets/left_shin.stl
- added link left_thigh, mass 0.606907; collision box size=0.0174299 0.0180598 0.058; collision box size=0.0224246 0.0239527 0.058
- added link part_1, mass 0.01458; visual mesh filename=package://assets/part_1.stl
- added link part_1_2, mass 0.01458; visual mesh filename=package://assets/part_1__2.stl
- added link right_arm, mass 0.121563; collision box size=0.0311265 0.205631 0.048; visual mesh filename=package://assets/right_arm.stl
- added link right_foot, mass 0.132264; collision box size=0.0399998 0.0101394 0.01; collision box size=0.0602786 0.0998323 0.01
- added link right_hand, mass 0.144242; collision box size=0.0286525 0.102703 0.041; collision cylinder length=0.041 radius=0.005
- added link right_shin, mass 0.36741; visual mesh filename=package://assets/right_shin.stl
- added link right_thigh, mass 0.596928; collision box size=0.0174297 0.0179047 0.058; collision box size=0.0224243 0.0224407 0.058
- link torso: mass 2.0839 -> 5.39548; geometry collision box size=0.0365497 0.0492657 0.026; collision box size=0.0365497 0.0492657 0.026
Joints:
- removed joint HeadPan
- removed joint HeadTilt
- removed joint LAnklePitch
- removed joint LAnkleRoll
- removed joint LElbow
- removed joint LHipPitch
- removed joint LHipRoll
- removed joint LHipYaw
- removed joint LKnee
- removed joint LLB
- removed joint LLF
- removed joint LRB
- removed joint LRF
- removed joint LShoulderPitch
- removed joint LShoulderRoll
- removed joint RAnklePitch
- removed joint RAnkleRoll
- removed joint RElbow
- removed joint RHipPitch
- removed joint RHipRoll
- removed joint RHipYaw
- removed joint RKnee
- removed joint RLB
- removed joint RLF
- removed joint RRB
- removed joint RRF
- removed joint RShoulderPitch
- removed joint RShoulderRoll
- removed joint base_link_to_base
- removed joint camera_frame
- removed joint camera_optical_frame_uncalibrated_frame
- removed joint imu_frame_2_frame
- removed joint imu_frame_uncalibrated_frame
- removed joint l_cleat_l_back_frame
- removed joint l_cleat_l_front_frame
- removed joint l_cleat_r_back_frame
- removed joint l_cleat_r_front_frame
- removed joint l_sole_frame
- removed joint l_toe_frame
- removed joint l_wrist_frame
- removed joint r_cleat_l_back_frame
- removed joint r_cleat_l_front_frame
- removed joint r_cleat_r_back_frame
- removed joint r_cleat_r_front_frame
- removed joint r_sole_frame
- removed joint r_toe_frame
- removed joint r_wrist_frame
- added joint arm_L_1: type revolute, parent torso, child part_1, origin xyz=-0.06405 -0.144944 0.119245 rpy=-1.5708 -4.46397e-16 -9.29758e-17, axis 0 0 1, limit lower=-2.26893 upper=2.26893 effort=10 velocity=10
- added joint arm_L_2: type revolute, parent part_1, child left_arm, origin xyz=0.020127 0.019 -0.022 rpy=-3.41096e-16 1.5708 0, axis 0 0 1, limit lower=-3.14159 upper=0.174533 effort=10 velocity=10
- added joint arm_L_3: type revolute, parent left_arm, child left_hand, origin xyz=-0.000234367 0.182 0.0012 rpy=-1.04777e-15 -2.6737e-16 -8.32668e-17, axis 0 0 1, limit lower=-1.5708 upper=1.5708 effort=10 velocity=10
- added joint arm_R_1: type revolute, parent torso, child part_1_2, origin xyz=-0.06405 0.148106 0.119245 rpy=-1.5708 -3.41792e-16 -3.14159, axis 0 0 1, limit lower=-2.35619 upper=2.35619 effort=10 velocity=10
- added joint arm_R_2: type revolute, parent part_1_2, child right_arm, origin xyz=-0.020127 0.019 -0.022 rpy=-1.17756e-14 -1.5708 0, axis 0 0 1, limit lower=-0.174533 upper=3.14159 effort=10 velocity=10
- added joint arm_R_3: type revolute, parent right_arm, child right_hand, origin xyz=-0.000456612 0.181999 0.0012 rpy=1.4988e-15 3.30449e-16 -7.24763e-24, axis 0 0 1, limit lower=-1.5708 upper=1.5708 effort=10 velocity=10
- added joint head_nod: type revolute, parent head_bottom, child head_top, origin xyz=0.02165 -8.05199e-11 -0.022 rpy=1.5708 -0.424601 1.5708, axis 0 0 1, limit lower=-1.5708 upper=1.0472 effort=10 velocity=10
- added joint head_turn: type revolute, parent torso, child head_bottom, origin xyz=-0.05035 0.0015808 0.160995 rpy=3.14159 -3.12214e-08 1.5708, axis 0 0 1, limit lower=-1.5708 upper=1.5708 effort=10 velocity=10
- added joint hip_left_x: type revolute, parent hip_left_z, child hip_left_x, origin xyz=2.60902e-15 -0.0225 -0.042 rpy=1.5708 7.76701e-15 8.12988e-14, axis 0 0 1, limit lower=-0.523599 upper=0.785398 effort=10 velocity=10
- added joint hip_left_z: type revolute, parent torso, child hip_left_z, origin xyz=-0.06405 0.0661808 -0.166455 rpy=1.20886e-14 -3.12214e-08 1.5708, axis 0 0 1, limit lower=-0.785398 upper=0.785398 effort=10 velocity=10
- added joint hip_right_x: type revolute, parent hip_right_z, child hip_right_x, origin xyz=1.59595e-15 -0.0225 -0.042 rpy=1.5708 7.99933e-15 6.43788e-14, axis 0 0 1, limit lower=-0.785398 upper=0.523599 effort=10 velocity=10
- added joint hip_right_z: type revolute, parent torso, child hip_right_z, origin xyz=-0.06405 -0.0629866 -0.166455 rpy=2.81209e-14 -3.12214e-08 1.5708, axis 0 0 1, limit lower=-0.785398 upper=0.785398 effort=10 velocity=10
- added joint left_foot_eversion: type revolute, parent 60645k191_ball_joint_rod_end_2, child left_foot, origin xyz=1.11022e-16 5.55112e-17 -1.38778e-17 rpy=-3.14159 1.5708 0, axis 0 0 1, limit lower=-0.523599 upper=0.523599 effort=10 velocity=10
- added joint left_foot_flexion: type revolute, parent left_shin, child 60645k191_ball_joint_rod_end_2, origin xyz=0.117972 -0.153164 -0.0051 rpy=-3.14159 -5.21728e-15 1.39626, axis 0 0 1, limit lower=0 upper=1.22173 effort=10 velocity=10
- added joint left_leg_raise: type revolute, parent hip_left_x, child left_thigh, origin xyz=-0.0051 -0.035 -0.0249827 rpy=-1.26083e-24 1.5708 0, axis 0 0 1, limit lower=-1.5708 upper=1.5708 effort=10 velocity=10
- added joint left_shin_extension: type revolute, parent left_thigh, child left_shin, origin xyz=1.84575e-15 -0.145716 0.0101 rpy=-6.87083e-15 8.51081e-17 -4.77077e-16, axis 0 0 1, limit lower=-1.0472 upper=1.5708 effort=10 velocity=10
- added joint right_foot_eversion: type revolute, parent 60645k191_ball_joint_rod_end, child right_foot, origin xyz=-5.55112e-17 5.55112e-17 0 rpy=2.69482e-17 1.5708 0, axis 0 0 1, limit lower=-0.523599 upper=0.523599 effort=10 velocity=10
- added joint right_foot_flexion: type revolute, parent right_shin, child 60645k191_ball_joint_rod_end, origin xyz=0.120398 -0.151264 -0.0049 rpy=3.14159 9.62969e-15 7.57809e-08, axis 0 0 1, limit lower=-1.22173 upper=7.10543e-15 effort=10 velocity=10
- added joint right_leg_raise: type revolute, parent hip_right_x, child right_thigh, origin xyz=0.0051 -0.035 -0.0249827 rpy=-3.14159 1.5708 0, axis 0 0 1, limit lower=-1.5708 upper=1.5708 effort=10 velocity=10
- added joint right_shin_extension: type revolute, parent right_thigh, child right_shin, origin xyz=-0.000786118 0.145714 0.0101 rpy=-6.6546e-15 -1.04807e-15 1.74533, axis 0 0 1, limit lower=-1.0472 upper=1.5708 effort=10 velocity=10
