Commit message: Fix pybullet simulation for Wolverbot URDF
- Add Wolverbot mesh assets to wolfgang_description and fix package:// paths
- Add base_link root to URDF so torso is discoverable as a non-root link
- Fix p.get_keyboardEvents() typo in simulation.py
- Wrap pybullet orientation tuple in np.array() for xyzw2wxyz() type requirement
- Fix pressure sensor guard to check per-robot dict; fix warn_once() -> warning()

File: urdf/robot.urdf (robot description, URDF)
Before this commit: robot maniskill, 22 links, 21 joints
Links:
- removed link base_link
- link ball_joint_rod_end: geometry visual mesh filename=package://assets/ball_joint_rod_end.stl
- link ball_joint_rod_end_2: geometry visual mesh filename=package://assets/ball_joint_rod_end.stl
- link head_bottom: geometry visual mesh filename=package://assets/head_bottom.stl
- link head_top: geometry visual mesh filename=package://assets/head_top.stl
- link hip_left_x: geometry visual mesh filename=package://assets/hip_left_x.stl
- link hip_left_z: geometry collision box size=0.0311905 0.00586106 0.034; collision box size=0.0317858 0.0071103 0.034
- link hip_right_x: geometry visual mesh filename=package://assets/hip_right_x.stl
- link hip_right_z: geometry collision box size=0.0311905 0.00586106 0.034; collision box size=0.0317858 0.0071103 0.034
- link left_arm: geometry collision box size=0.029846 0.205415 0.048; visual mesh filename=package://assets/left_arm.stl
- link left_foot: geometry collision box size=0.0399948 0.0108051 0.01; collision box size=0.061605 0.0990193 0.01
- link left_hand: geometry collision box size=0.0319403 0.0740559 0.041; collision box size=0.032 0.0302663 0.041
- link left_shin: geometry visual mesh filename=package://assets/left_shin.stl
- link left_thigh: geometry collision box size=0.0174299 0.0180598 0.058; collision box size=0.0224246 0.0239527 0.058
- link part_1: geometry visual mesh filename=package://assets/part_1.stl
- link part_1_2: geometry visual mesh filename=package://assets/part_1__2.stl
- link right_arm: geometry collision box size=0.0311265 0.205631 0.048; visual mesh filename=package://assets/right_arm.stl
- link right_foot: geometry collision box size=0.0399998 0.0101394 0.01; collision box size=0.0602786 0.0998323 0.01
- link right_hand: geometry collision box size=0.0286525 0.102703 0.041; collision cylinder length=0.041 radius=0.005
- link right_shin: geometry visual mesh filename=package://assets/right_shin.stl
- link right_thigh: geometry collision box size=0.0174297 0.0179047 0.058; collision box size=0.0224243 0.0224407 0.058
- link torso: geometry collision box size=0.0365497 0.0492657 0.026; collision box size=0.0365497 0.0492657 0.026
Joints:
- removed joint base_link_to_base
